File: BLDC_DRIVER/Motor_driver.kicad_sch (KiCad schematic)
At the start: 54 parts, among them IC2 DRV8323SRTAR, Q1 SQJ170ELP, Q2 SQJ170ELP, Q3 SQJ170ELP, Q4 SQJ170ELP, Q5 SQJ170ELP, Q6 SQJ170ELP

Commit message: added footprints, fault detection and temperature calc
Parts:
- removed C24: 100n, symbol Device:C
- removed D4, D5, D6, D7: TODO, symbol Device:D_Schottky
- removed R22: 34.8k, symbol Device:R
- removed R23: 4.99k, symbol Device:R
- added C104: 100u/200V, EMVY101ARA101MKE0S:CAPAE1300X1400N, symbol Device:C_Polarized
- added C109: 10u/100V, Capacitor_SMD:C_1210_3225Metric, symbol Device:C
- added C110: 100n/200V, Capacitor_SMD:C_0805_2012Metric, symbol Device:C
- added C112: 1u, Capacitor_SMD:C_0805_2012Metric, symbol Device:C
- added C116, C119, C120, C121, C131, C132: 10n/200V, Capacitor_SMD:C_0805_2012Metric, symbol Device:C
- added C125: 100n, Capacitor_SMD:C_0603_1608Metric, symbol Device:C
- added C126: 1n, Capacitor_SMD:C_0603_1608Metric, symbol Device:C
- added D101, D102, D103, D104, D105, D106: RF201L2SDDTE25, RF201L2SDDTE25:DIOM5026X220N, symbol RF201L2SDDTE25:RF201L2SDDTE25
- added D107, D108, D110, D111, D112: BAT54C, Package_TO_SOT_SMD:SOT-23, symbol Diode:BAT54C
- added L101: 1u/30A, PM4343.102NLT:INDPM140128X650N, symbol PM4343_102NLT:PM4343.102NLT
- added R105, R106, R107, R111, R112, R113: 10R, Resistor_SMD:R_1210_3225Metric, symbol Device:R
- added R120: 10k, Resistor_SMD:R_0603_1608Metric, symbol Device:R
- added R121: 34.8k, Resistor_SMD:R_0603_1608Metric, symbol Device:R
- added R126: 4.99k, Resistor_SMD:R_0603_1608Metric, symbol Device:R
- added TH101: 47k, Resistor_SMD:R_0603_1608Metric, symbol Device:Thermistor_NTC
- added TP101, TP102, TP103, TP104, TP105, TP106, TP107, TP108, TP109, TP110, TP111, TP112, TP113, TP114, TP115, TP116, TP117, TP118, TP119, TP120, TP121, TP122, TP123, TP124, TP125: TestPoint, TestPoint:TestPoint_Pad_D2.5mm, symbol Connector:TestPoint
- C101: renamed from C29; value 1u -> 1u/6.3V; footprint (none) -> Capacitor_SMD:C_0603_1608Metric
- C102: renamed from C23; value 10n -> 10n/200V; footprint (none) -> Capacitor_SMD:C_0805_2012Metric
- C103: renamed from C20; value 220u -> 100u/200V; footprint (none) -> EMVY101ARA101MKE0S:CAPAE1300X1400N
- C105: renamed from C21; value 220u -> 100u/200V; footprint (none) -> EMVY101ARA101MKE0S:CAPAE1300X1400N
- C106: renamed from C22; value 220u -> 100u/200V; footprint (none) -> EMVY101ARA101MKE0S:CAPAE1300X1400N
- C107: renamed from C13; value 47n -> 47n/200V; footprint (none) -> Capacitor_SMD:C_0805_2012Metric
- C108: renamed from C17; value 1u -> 1u/16V; footprint (none) -> Capacitor_SMD:C_0805_2012Metric
- C111: renamed from C30; footprint (none) -> Capacitor_SMD:C_0603_1608Metric
- C113: renamed from C18; footprint (none) -> Capacitor_SMD:C_1206_3216Metric
- C114: renamed from C16; footprint (none) -> Capacitor_SMD:C_1206_3216Metric
- C115: renamed from C19; footprint (none) -> Capacitor_SMD:C_1206_3216Metric
- C122: renamed from C14; footprint (none) -> Capacitor_SMD:C_0603_1608Metric
- C123: renamed from C15; footprint (none) -> Capacitor_SMD:C_0603_1608Metric
- C124: renamed from C12; footprint (none) -> Capacitor_SMD:C_0603_1608Metric
- C127: renamed from C26; footprint (none) -> Capacitor_SMD:C_0603_1608Metric
- C128: renamed from C27; footprint (none) -> Capacitor_SMD:C_0603_1608Metric
- C129: renamed from C28; footprint (none) -> Capacitor_SMD:C_0603_1608Metric
- C130: renamed from C25; footprint (none) -> Capacitor_SMD:C_0603_1608Metric
- IC101: renamed from IC2; footprint QFN50P600X600X80-41N-D -> DRV8323:QFN50P600X600X80-41N-D
- Q101: renamed from Q3; footprint SQJ160EPT1_GE3 -> SQJ170ELP-T1_GE3:SQJ160EPT1_GE3
- Q102: renamed from Q5; footprint SQJ160EPT1_GE3 -> SQJ170ELP-T1_GE3:SQJ160EPT1_GE3
- Q103: renamed from Q1; footprint SQJ160EPT1_GE3 -> SQJ170ELP-T1_GE3:SQJ160EPT1_GE3
- Q104: renamed from Q4; footprint SQJ160EPT1_GE3 -> SQJ170ELP-T1_GE3:SQJ160EPT1_GE3
- Q105: renamed from Q6; footprint SQJ160EPT1_GE3 -> SQJ170ELP-T1_GE3:SQJ160EPT1_GE3
- Q106: renamed from Q2; footprint SQJ160EPT1_GE3 -> SQJ170ELP-T1_GE3:SQJ160EPT1_GE3
- R101: renamed from R33; value 0R -> 0R/2W; footprint (none) -> Resistor_SMD:R_2010_5025Metric
- R102: renamed from R21; footprint (none) -> Resistor_SMD:R_2010_5025Metric
- R103: renamed from R34; footprint (none) -> Resistor_SMD:R_0603_1608Metric
- R104: renamed from R35; footprint (none) -> Resistor_SMD:R_0603_1608Metric
- R108: renamed from R11; value 10R -> 1R; footprint (none) -> Resistor_SMD:R_1210_3225Metric
- R109: renamed from R16; value 10R -> 1R; footprint (none) -> Resistor_SMD:R_1210_3225Metric
- R110: renamed from R6; value 10R -> 1R; footprint (none) -> Resistor_SMD:R_1210_3225Metric
- R114: renamed from R12; value 10R -> 1R; footprint (none) -> Resistor_SMD:R_1210_3225Metric
- R115: renamed from R17; value 10R -> 1R; footprint (none) -> Resistor_SMD:R_1210_3225Metric
- R116: renamed from R7; value 10R -> 1R; footprint (none) -> Resistor_SMD:R_1210_3225Metric
- R117: renamed from R13; footprint (none) -> Resistor_SMD:R_2512_6332Metric
- R118: renamed from R18; footprint (none) -> Resistor_SMD:R_2512_6332Metric
- R119: renamed from R8; footprint (none) -> Resistor_SMD:R_2512_6332Metric
- R122: renamed from R24; footprint (none) -> Resistor_SMD:R_0603_1608Metric
- R123: renamed from R27; footprint (none) -> Resistor_SMD:R_0603_1608Metric
- R124: renamed from R25; footprint (none) -> Resistor_SMD:R_0603_1608Metric
- R125: renamed from R28; footprint (none) -> Resistor_SMD:R_0603_1608Metric
- R127: renamed from R26; footprint (none) -> Resistor_SMD:R_0603_1608Metric
- R128: renamed from R29; footprint (none) -> Resistor_SMD:R_0603_1608Metric
- R129: renamed from R30; footprint (none) -> Resistor_SMD:R_0603_1608Metric
- R130: renamed from R31; footprint (none) -> Resistor_SMD:R_0603_1608Metric
- R131: renamed from R32; footprint (none) -> Resistor_SMD:R_0603_1608Metric
Connections:
- net +3.3V: now also C112.1, R120.1
- net +48V: now also L101.1; no longer C102.1, C105.1, C106.1, C108.1, C113.1, C114.1, C115.1, IC101.4 (VM), IC101.5 (VDRAIN), Q101.9, Q102.9, Q103.9
- net GHA: now also D103.1 (K)
- net GHB: now also D101.1 (K)
- net GHC: now also D102.1 (K)
- net GLA: now also D106.1 (K)
- net GLB: now also D104.1 (K)
- net GLC: now also D105.1 (K)
- net GND: now also IC101.10 (SNA), IC101.11 (SNB), IC101.20 (SNC), C104.2, C109.2, C110.2, C112.2, C125.2, C126.2, R126.2, TH101.2; no longer IC101.12 (SPB), IC101.19 (SPC), IC101.9 (SPA)
- net PVDDSENSE: now also C125.1, D110.1, R121.2, R126.1, TP121.1
- net SHA: now also C121.2, R113.1, TP109.1, TP110.1
- net SHB: now also C116.2, R111.1, TP105.1, TP106.1
- net SHC: now also C120.2, R112.1, TP107.1, TP108.1
- net SLA: now also IC101.9 (SPA), C131.2, TP116.1, TP119.1; no longer IC101.10 (SNA)
- net SLB: now also IC101.12 (SPB), C119.2, TP114.1, TP117.1; no longer IC101.11 (SNB)
- net SLC: now also IC101.19 (SPC), C132.2, TP115.1, TP118.1; no longer IC101.20 (SNC)
- net SensIA: now also D111.2
- net SensIB: now also D111.1
- net SensIC: now also D112.1
- net SensVA: now also D107.2, TP122.1
- net SensVB: now also D107.1, TP123.1
- net SensVC: now also D108.2, TP124.1
- net SensVN: now also D108.1, TP120.1
- net at Q105.4, R115.2: now also D105.2 (A), TP112.1
- net at Q101.4, R108.2: now also D101.2 (A), TP102.1
- net at Q103.4, R110.2: now also D103.2 (A), TP104.1
- net at Q102.4, R109.2: now also D102.2 (A), TP103.1
- net at Q106.4, R116.2: now also D106.2 (A), TP113.1
- net at Q104.4, R114.2: now also D104.2 (A), TP111.1
- new net: C116.1, R105.2
- new net: C120.1, R106.2
- new net: C121.1, R107.2
- new net: C132.1, R112.2
- new net: C131.1, R113.2
- new net: C119.1, R111.2
- new net TEMP_MOSFET: C126.1, D110.2, R120.2, TH101.1, TP125.1
- new net Vdrive: C102.1, C104.1, C105.1, C106.1, C108.1, C109.1, C110.1, C113.1, C114.1, C115.1, IC101.4 (VM), IC101.5 (VDRAIN), L101.2, Q101.9, Q102.9, Q103.9, R105.1, R106.1, R107.1, R121.1, TP101.1
- no-connect marks 0 -> 1
Other:
- note added: "Fault detection / protection"
- note added: "Half bridge, short loop as possible"
- note added: "X7R near IC"
- note added: "far from half bridge"
- note added: "near IC"
- note added: "near half bridge"
- note removed: "Half bridge"
- moved on the sheet: C101, C102, C103, C105, C106, C107, C108, C111, C113, C114, C115, C122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

Commit message: snuber, removing spice
Parts:
- removed C116: 10n/200V, Capacitor_SMD:C_0805_2012Metric, symbol Device:C
- removed R105, R106: 10R, Resistor_SMD:R_1210_3225Metric, symbol Device:R
- removed TP105, TP107, TP109: TestPoint, TestPoint:TestPoint_Pad_D2.5mm, symbol Connector:TestPoint
- added C131: 10n/200V, Capacitor_SMD:C_0805_2012Metric, symbol Device:C
- added D112, D113, D114, D115, D116, D117: RF201L2SDDTE25, RF201L2SDDTE25:DIOM5026X220N, symbol RF201L2SDDTE25:RF201L2SDDTE25
- added R118, R120, R122: 20m, Resistor_SMD:R_2512_6332Metric, symbol Device:R
- added R135, R136: 10R, Resistor_SMD:R_1210_3225Metric, symbol Device:R
- R117: value 10m -> 20m
- R119: renamed from R118; value 10m -> 20m
- R121: renamed from R119; value 10m -> 20m
- renumbered C121 to C118, C131 to C121, D110 to D109, D111 to D110, D112 to D111, R120 to R123, R121 to R124, R122 to R125, R123 to R126, R124 to R127, R125 to R128, R126 to R129, R127 to R130, R128 to R131, R129 to R132, R130 to R133, R131 to R134, TP121 to TP120, TP120 to TP121
Connections:
- net +3.3V: now also D107.3, D108.3, D109.3, D110.3, D111.3
- net GND: now also R118.2, R120.2, R122.2
- net SHA: now also D112.1 (K), D113.2 (A); no longer C118.2, R113.1
- net SHB: now also D114.1 (K), D115.2 (A); no longer R111.1
- net SHC: now also D116.1 (K), D117.2 (A); no longer C120.2, R112.1
- net SLA: now also R107.2, R122.1
- net SLB: now also R111.2, C131.2, R118.1; no longer C119.2
- net SLC: now also R112.2, R120.1
- net Vdrive: now also C118.1, C119.1, C120.1, R113.1, R135.1, R136.1; no longer R107.1
- net at C132.1: now also D117.1 (K), R136.2; no longer R112.2
- net at C121.1, R113.2: now also D113.1 (K)
- new net: C118.2, D112.2 (A), R107.1
- new net: C120.2, D116.2 (A), R112.1
- new net: C119.2, D114.2 (A), R111.1
- new net: C131.1, D115.1 (K), R135.2
Other:
- moved on the sheet: C118, C121, R107, R113, TP106, TP108, TP110
