File: BLDC_DRIVER/BLDC_DRIVER.kicad_pcb (KiCad board)
At the start: 2 copper layers, 0 parts

Commit message: finall motor driver
Parts:
- added C1: 10uF, EMVY101ARA101MKE0S:CAPAE1300X1400N, F.Cu at (134.7, 153.0)
- added C10: 100nF, Capacitor_SMD:C_0805_2012Metric_Pad1.18x1.45mm_HandSolder, F.Cu at (106.0, 164.9)
- added C101: 1u/6.3V, Capacitor_SMD:C_0603_1608Metric, F.Cu at (73.2, 52.4)
- added C103: 100u/200V, EMVY101ARA101MKE0S:CAPAE1300X1400N, F.Cu at (28.6, 24.2)
- added C104: 220u/63V, EMVY101ARA101MKE0S:CAPAE1300X1400N, F.Cu at (28.6, 39.5)
- added C105: 100u/200V, EMVY101ARA101MKE0S:CAPAE1300X1400N, F.Cu at (28.6, 54.7)
- added C106: 100u/200V, EMVY101ARA101MKE0S:CAPAE1300X1400N, F.Cu at (28.6, 70.0)
- added C107: 47n/200V, Capacitor_SMD:C_0805_2012Metric, F.Cu at (82.0, 37.6)
- added C108: 1u/16V, Capacitor_SMD:C_0805_2012Metric, F.Cu at (82.0, 40.6)
- added C109: 10u/100V, Capacitor_SMD:C_1210_3225Metric, F.Cu at (59.8, 74.6)
- added C11: 10u, Capacitor_SMD:C_0603_1608Metric_Pad1.08x0.95mm_HandSolder, F.Cu at (30.9, 151.5)
- added C110: 100n/200V, Capacitor_SMD:C_0805_2012Metric, F.Cu at (82.0, 43.6)
- added C111: 100n, Capacitor_SMD:C_0603_1608Metric, F.Cu at (73.2, 54.9)
- added C112: 1u, Capacitor_SMD:C_0805_2012Metric, F.Cu at (82.0, 46.6)
- added C113: 10u, Capacitor_SMD:C_1206_3216Metric, F.Cu at (65.7, 37.8)
- added C114: 10u, Capacitor_SMD:C_1206_3216Metric, F.Cu at (65.7, 41.1)
- added C115: 10u, Capacitor_SMD:C_1206_3216Metric, F.Cu at (65.7, 44.5)
- added C116: 10u, Capacitor_SMD:C_1206_3216Metric, F.Cu at (65.7, 47.8)
- added C117: 10u, Capacitor_SMD:C_1206_3216Metric, F.Cu at (71.3, 37.8)
- added C118: 10n/200V, Capacitor_SMD:C_1206_3216Metric, F.Cu at (71.3, 41.1)
- added C119: 10n/200V, Capacitor_SMD:C_1206_3216Metric, F.Cu at (71.3, 44.5)
- added C12: 100n, Capacitor_SMD:C_0603_1608Metric_Pad1.08x0.95mm_HandSolder, F.Cu at (30.9, 154.0)
- added C120: 10n/200V, Capacitor_SMD:C_1206_3216Metric, F.Cu at (71.3, 47.8)
- added C121: 10n/200V, Capacitor_SMD:C_1206_3216Metric, F.Cu at (77.0, 37.8)
- added C122: 1n, Capacitor_SMD:C_0603_1608Metric, F.Cu at (73.2, 57.4)
- added C123: 1n, Capacitor_SMD:C_0603_1608Metric, F.Cu at (73.2, 59.9)
- added C124: 1n, Capacitor_SMD:C_0603_1608Metric, F.Cu at (73.2, 62.5)
- added C125: 100n, Capacitor_SMD:C_0603_1608Metric, F.Cu at (73.2, 65.0)
- added C126: 1n, Capacitor_SMD:C_0603_1608Metric, F.Cu at (73.2, 67.5)
- added C127: 1n, Capacitor_SMD:C_0603_1608Metric, F.Cu at (77.2, 52.4)
- added C128: 1n, Capacitor_SMD:C_0603_1608Metric, F.Cu at (77.2, 54.9)
- added C129: 1n, Capacitor_SMD:C_0603_1608Metric, F.Cu at (77.2, 57.4)
- added C13: 100n, Capacitor_SMD:C_0603_1608Metric_Pad1.08x0.95mm_HandSolder, F.Cu at (30.9, 156.6)
- added C130: 1n, Capacitor_SMD:C_0603_1608Metric, F.Cu at (77.2, 59.9)
- added C131: 10n/200V, Capacitor_SMD:C_1206_3216Metric, F.Cu at (77.0, 41.1)
- added C132: 10n/200V, Capacitor_SMD:C_1206_3216Metric, F.Cu at (77.0, 44.5)
- added C133: 10u, Capacitor_SMD:C_1206_3216Metric, F.Cu at (77.0, 47.8)
- added C134: 10n/200V, Capacitor_SMD:C_0805_2012Metric, F.Cu at (82.0, 49.6)
- added C135: 10u/100V, Capacitor_SMD:C_1210_3225Metric, F.Cu at (59.8, 78.8)
- added C14: 100n, Capacitor_SMD:C_0603_1608Metric_Pad1.08x0.95mm_HandSolder, F.Cu at (30.9, 159.1)
- added C15: 10u, Capacitor_SMD:C_0603_1608Metric_Pad1.08x0.95mm_HandSolder, F.Cu at (30.9, 161.6)
- added C16: 12p, Capacitor_SMD:C_0603_1608Metric_Pad1.08x0.95mm_HandSolder, F.Cu at (30.9, 164.1)
- added C17: 12p, Capacitor_SMD:C_0603_1608Metric_Pad1.08x0.95mm_HandSolder, F.Cu at (30.9, 166.6)
- added C18: 100n, Capacitor_SMD:C_0603_1608Metric_Pad1.08x0.95mm_HandSolder, F.Cu at (35.2, 151.5)
- added C19: 100n, Capacitor_SMD:C_0603_1608Metric_Pad1.08x0.95mm_HandSolder, F.Cu at (35.2, 154.0)
- added C2: 1uF, Capacitor_SMD:C_0805_2012Metric_Pad1.18x1.45mm_HandSolder, F.Cu at (106.0, 146.9)
- added C20: 100n, Capacitor_SMD:C_0603_1608Metric_Pad1.08x0.95mm_HandSolder, F.Cu at (35.2, 156.6)
- added C21: 10u, Capacitor_SMD:C_0603_1608Metric_Pad1.08x0.95mm_HandSolder, F.Cu at (35.2, 159.1)
- added C22: 100n, Capacitor_SMD:C_0603_1608Metric_Pad1.08x0.95mm_HandSolder, F.Cu at (35.2, 161.6)
- added C23: 100n, Capacitor_SMD:C_0603_1608Metric_Pad1.08x0.95mm_HandSolder, F.Cu at (35.2, 164.1)
- added C3: 100nF, Capacitor_SMD:C_0805_2012Metric_Pad1.18x1.45mm_HandSolder, F.Cu at (106.0, 149.9)
- added C4: 100nF, Capacitor_SMD:C_0603_1608Metric_Pad1.08x0.95mm_HandSolder, F.Cu at (127.3, 131.5)
- added C5: 10uF, Capacitor_SMD:C_0805_2012Metric_Pad1.18x1.45mm_HandSolder, F.Cu at (106.0, 152.9)
- added C6: 1uF, Capacitor_SMD:C_0805_2012Metric_Pad1.18x1.45mm_HandSolder, F.Cu at (106.0, 155.9)
- added C7: 10uF, Capacitor_SMD:C_0805_2012Metric_Pad1.18x1.45mm_HandSolder, F.Cu at (106.0, 158.9)
- added C8: 100n, Capacitor_SMD:C_0603_1608Metric_Pad1.08x0.95mm_HandSolder, F.Cu at (127.3, 134.0)
- added C9: 22uF, Capacitor_SMD:C_0805_2012Metric_Pad1.18x1.45mm_HandSolder, F.Cu at (106.0, 161.9)
- added D1: D_Schottky, Diode_SMD:D_SMA, F.Cu at (133.6, 140.9)
- added D101: SBR3U60P1-7, Diode_SMD:D_PowerDI-123, F.Cu at (53.9, 53.0)
- added D102: SBR3U60P1-7, Diode_SMD:D_PowerDI-123, F.Cu at (53.9, 56.6)
- added D103: SBR3U60P1-7, Diode_SMD:D_PowerDI-123, F.Cu at (53.9, 60.3)
- added D104: SBR3U60P1-7, Diode_SMD:D_PowerDI-123, F.Cu at (53.9, 63.9)
- added D105: SBR3U60P1-7, Diode_SMD:D_PowerDI-123, F.Cu at (53.9, 67.6)
- added D106: SBR3U60P1-7, Diode_SMD:D_PowerDI-123, F.Cu at (53.9, 71.2)
- added D107: BAT54C, Package_TO_SOT_SMD:SOT-23, F.Cu at (48.5, 53.6)
- added D108: BAT54C, Package_TO_SOT_SMD:SOT-23, F.Cu at (48.5, 58.2)
- added D109: BAT54C, Package_TO_SOT_SMD:SOT-23, F.Cu at (48.5, 62.8)
- added D110: BAT54C, Package_TO_SOT_SMD:SOT-23, F.Cu at (48.5, 67.4)
- added D111: BAT54C, Package_TO_SOT_SMD:SOT-23, F.Cu at (48.5, 72.1)
- added D2: LED, Diode_SMD:D_0805_2012Metric_Pad1.15x1.40mm_HandSolder, F.Cu at (57.2, 161.5)
- added D3: LED, Diode_SMD:D_0805_2012Metric_Pad1.15x1.40mm_HandSolder, F.Cu at (57.2, 164.5)
- added D4: LED, Diode_SMD:D_0805_2012Metric_Pad1.15x1.40mm_HandSolder, F.Cu at (57.2, 167.6)
- added F1: 15A, Fuse:Fuse_Blade_ATO_directSolder, F.Cu at (109.7, 134.1)
- added F2: 15A, Fuse:Fuse_Blade_ATO_directSolder, F.Cu at (109.7, 141.6)
- added FB1: FerriteBead, Inductor_SMD:L_0805_2012Metric_Pad1.05x1.20mm_HandSolder, F.Cu at (57.9, 144.8)
- added IC101: DRV8323SRTAR, DRV8323:QFN50P600X600X80-41N-D, F.Cu at (41.5, 59.4)
- added J1: XT60, Connector_AMASS:AMASS_XT60-M_1x02_P7.20mm_Vertical, F.Cu at (113.6, 150.5)
- added J104: 691311400103, 691311400103:691311400103, F.Cu at (75.1, 31.4)
- added J2: Conn_01x03_Pin, Connector_PinHeader_2.54mm:PinHeader_1x03_P2.54mm_Vertical, F.Cu at (57.1, 152.6)
- added J3: Conn_01x03_Pin, Connector_PinHeader_2.54mm:PinHeader_1x03_P2.54mm_Vertical, F.Cu at (61.7, 152.6)
- added J4: Conn_01x06_Pin, Connector_PinHeader_2.54mm:PinHeader_1x06_P2.54mm_Vertical, F.Cu at (48.4, 152.6)
- added JP1: Jumper_2_Bridged, Jumper:SolderJumper-2_P1.3mm_Open_TrianglePad1.0x1.5mm, F.Cu at (61.7, 161.8)
- added JP2: Jumper_2_Bridged, Jumper:SolderJumper-2_P1.3mm_Open_TrianglePad1.0x1.5mm, F.Cu at (61.7, 165.3)
- added L1: 15uH, Inductor_SMD:L_APV_ANR6045, F.Cu at (112.3, 159.4)
- added Q101: BSC146N10LS5ATMA1, BSC146N10LS5ATMA1:BSC146N10LS5ATMA1, F.Cu at (40.9, 20.9)
- added Q102: BSC146N10LS5ATMA1, BSC146N10LS5ATMA1:BSC146N10LS5ATMA1, F.Cu at (48.2, 20.9)
- added Q103: BSC146N10LS5ATMA1, BSC146N10LS5ATMA1:BSC146N10LS5ATMA1, F.Cu at (55.4, 20.9)
- added Q104: BSC146N10LS5ATMA1, BSC146N10LS5ATMA1:BSC146N10LS5ATMA1, F.Cu at (62.7, 20.9)
- added Q105: BSC146N10LS5ATMA1, BSC146N10LS5ATMA1:BSC146N10LS5ATMA1, F.Cu at (69.9, 20.9)
- added Q106: BSC146N10LS5ATMA1, BSC146N10LS5ATMA1:BSC146N10LS5ATMA1, F.Cu at (77.2, 20.9)
- added R1: R, Resistor_SMD:R_0603_1608Metric_Pad0.98x0.95mm_HandSolder, F.Cu at (127.3, 136.6)
- added R10: 4.7k, Resistor_SMD:R_0603_1608Metric, F.Cu at (52.8, 156.6)
- added R101: 0R/2W, Resistor_SMD:R_2010_5025Metric, F.Cu at (66.3, 74.6)
- added R103: 10k, Resistor_SMD:R_0603_1608Metric, F.Cu at (77.2, 62.5)
- added R104: 10k, Resistor_SMD:R_0603_1608Metric, F.Cu at (77.2, 65.0)
- added R105: 3.3R, Resistor_SMD:R_2010_5025Metric, F.Cu at (66.3, 78.8)
- added R107: 10R, Resistor_SMD:R_1210_3225Metric, F.Cu at (48.8, 28.0)
- added R108: 1R, Resistor_SMD:R_1210_3225Metric, F.Cu at (48.8, 32.2)
- added R109: 1R, Resistor_SMD:R_1210_3225Metric, F.Cu at (48.8, 36.4)
- added R11: 4.7k, Resistor_SMD:R_0603_1608Metric, F.Cu at (52.8, 159.1)
- added R110: 10R, Resistor_SMD:R_1210_3225Metric, F.Cu at (48.8, 40.6)
- added R111: 10R, Resistor_SMD:R_1210_3225Metric, F.Cu at (48.8, 44.8)
- added R112: 10R, Resistor_SMD:R_1210_3225Metric, F.Cu at (48.8, 49.0)
- added R113: 10R, Resistor_SMD:R_1210_3225Metric, F.Cu at (54.4, 28.0)
- added R114: 1R, Resistor_SMD:R_1210_3225Metric, F.Cu at (54.4, 32.2)
- added R115: 1R, Resistor_SMD:R_1210_3225Metric, F.Cu at (54.4, 36.4)
- added R116: 1R, Resistor_SMD:R_1210_3225Metric, F.Cu at (54.4, 40.6)
- added R117: 20m, Resistor_SMD:R_2512_6332Metric, F.Cu at (41.7, 28.3)
- added R118: 20m, Resistor_SMD:R_2512_6332Metric, F.Cu at (41.7, 33.2)
- added R119: 20m, Resistor_SMD:R_2512_6332Metric, F.Cu at (41.7, 38.1)
- added R12: 4.7k, Resistor_SMD:R_0603_1608Metric_Pad0.98x0.95mm_HandSolder, F.Cu at (39.6, 156.6)
- added R120: 20m, Resistor_SMD:R_2512_6332Metric, F.Cu at (41.7, 43.0)
- added R121: 20m, Resistor_SMD:R_2512_6332Metric, F.Cu at (41.7, 47.9)
- added R122: 20m, Resistor_SMD:R_2512_6332Metric, F.Cu at (41.7, 52.8)
- added R123: 10k, Resistor_SMD:R_0603_1608Metric, F.Cu at (77.2, 67.5)
- added R124: 34.8k, Resistor_SMD:R_0603_1608Metric, F.Cu at (81.2, 52.4)
- added R125: 47k, Resistor_SMD:R_0603_1608Metric, F.Cu at (81.2, 54.9)
- added R126: 47k, Resistor_SMD:R_0603_1608Metric, F.Cu at (81.2, 57.4)
- added R127: 47k, Resistor_SMD:R_0603_1608Metric, F.Cu at (81.2, 59.9)
- added R128: 47k, Resistor_SMD:R_0603_1608Metric, F.Cu at (81.2, 62.5)
- added R129: 4.99k, Resistor_SMD:R_0603_1608Metric, F.Cu at (81.2, 65.0)
- added R13: 10k, Resistor_SMD:R_0603_1608Metric_Pad0.98x0.95mm_HandSolder, F.Cu at (39.6, 159.1)
- added R130: 47k, Resistor_SMD:R_0603_1608Metric, F.Cu at (81.2, 67.5)
- added R131: 47k, Resistor_SMD:R_0603_1608Metric, F.Cu at (85.2, 52.4)
- added R132: 10k, Resistor_SMD:R_0603_1608Metric, F.Cu at (85.2, 54.9)
- added R133: 10k, Resistor_SMD:R_0603_1608Metric, F.Cu at (85.2, 57.4)
- added R134: 10k, Resistor_SMD:R_0603_1608Metric, F.Cu at (85.2, 59.9)
- added R135: 10R, Resistor_SMD:R_1210_3225Metric, F.Cu at (54.4, 44.8)
- added R136: 10R, Resistor_SMD:R_1210_3225Metric, F.Cu at (54.4, 49.0)
- added R137: 1R, Resistor_SMD:R_1210_3225Metric, F.Cu at (60.0, 28.0)
- added R138: 10R, Resistor_SMD:R_1210_3225Metric, F.Cu at (60.0, 32.2)
- added R139: 10R, Resistor_SMD:R_1210_3225Metric, F.Cu at (60.0, 36.4)
- added R14: 10k, Resistor_SMD:R_0603_1608Metric_Pad0.98x0.95mm_HandSolder, F.Cu at (39.6, 161.6)
- added R140: 10R, Resistor_SMD:R_1210_3225Metric, F.Cu at (60.0, 40.6)
- added R141: 10R, Resistor_SMD:R_1210_3225Metric, F.Cu at (60.0, 44.8)
- added R142: 10R, Resistor_SMD:R_1210_3225Metric, F.Cu at (60.0, 49.0)
- added R15: 4.7k, Resistor_SMD:R_0603_1608Metric_Pad0.98x0.95mm_HandSolder, F.Cu at (39.6, 164.1)
- added R16: 4.7k, Resistor_SMD:R_0603_1608Metric_Pad0.98x0.95mm_HandSolder, F.Cu at (39.6, 166.6)
- added R17: 4.7k, Resistor_SMD:R_0603_1608Metric_Pad0.98x0.95mm_HandSolder, F.Cu at (43.9, 151.5)
- added R18: 4.7k, Resistor_SMD:R_0603_1608Metric_Pad0.98x0.95mm_HandSolder, F.Cu at (43.9, 154.0)
- added R19: 10k, Resistor_SMD:R_0603_1608Metric_Pad0.98x0.95mm_HandSolder, F.Cu at (43.9, 156.6)
- added R2: R, Resistor_SMD:R_0603_1608Metric_Pad0.98x0.95mm_HandSolder, F.Cu at (127.3, 139.1)
- added R20: 10k, Resistor_SMD:R_0603_1608Metric_Pad0.98x0.95mm_HandSolder, F.Cu at (43.9, 159.1)
- added R21: 4.7k, Resistor_SMD:R_0603_1608Metric_Pad0.98x0.95mm_HandSolder, F.Cu at (43.9, 161.6)
- added R22: 4.7k, Resistor_SMD:R_0603_1608Metric_Pad0.98x0.95mm_HandSolder, F.Cu at (43.9, 164.1)
- added R3: 116k, Resistor_SMD:R_0603_1608Metric_Pad0.98x0.95mm_HandSolder, F.Cu at (127.3, 141.6)
- added R4: 22.1k, Resistor_SMD:R_0603_1608Metric_Pad0.98x0.95mm_HandSolder, F.Cu at (127.3, 144.1)
- added R5: 4.7k, Resistor_SMD:R_0603_1608Metric_Pad0.98x0.95mm_HandSolder, F.Cu at (35.2, 166.6)
- added R6: 4.7k, Resistor_SMD:R_0603_1608Metric_Pad0.98x0.95mm_HandSolder, F.Cu at (39.6, 151.5)
- added R7: 4.7k, Resistor_SMD:R_0603_1608Metric_Pad0.98x0.95mm_HandSolder, F.Cu at (39.6, 154.0)
- added R8: 4.7k, Resistor_SMD:R_0603_1608Metric, F.Cu at (52.8, 151.5)
- added R9: 4.7k, Resistor_SMD:R_0603_1608Metric, F.Cu at (52.8, 154.0)
- added SW1: SW_Push_Dual_x2, Button_Switch_SMD:SW_Push_1P1T_NO_CK_KSC7xxJ, F.Cu at (23.6, 132.9)
- added SW2: SW_Push_Dual_x2, Button_Switch_SMD:SW_Push_1P1T_NO_CK_KSC7xxJ, F.Cu at (23.6, 140.7)
- added SW3: SW_Push_Dual_x2, Button_Switch_SMD:SW_Push_1P1T_NO_CK_KSC7xxJ, F.Cu at (23.6, 148.4)
- added SW4: SW_Push_Dual_x2, Button_Switch_SMD:SW_Push_1P1T_NO_CK_KSC7xxJ, F.Cu at (23.6, 156.2)
- added SW5: SW_Push_Dual_x2, Button_Switch_SMD:SW_Push_1P1T_NO_CK_KSC7xxJ, F.Cu at (23.6, 163.9)
- added TH101: 47k, Resistor_SMD:R_0603_1608Metric, F.Cu at (85.2, 62.5)
- added TP1: TestPoint, TestPoint:TestPoint_Pad_D1.5mm, F.Cu at (117.9, 157.4)
- added TP101: TestPoint, TestPoint:TestPoint_Pad_D1.5mm, F.Cu at (2.80, 46.9)
- added TP102: TestPoint, TestPoint:TestPoint_Pad_D1.5mm, F.Cu at (2.80, 50.5)
- added TP103: TestPoint, TestPoint:TestPoint_Pad_D1.5mm, F.Cu at (2.80, 54.0)
- added TP104: TestPoint, TestPoint:TestPoint_Pad_D1.5mm, F.Cu at (2.80, 57.5)
- added TP106: TestPoint, TestPoint:TestPoint_Pad_D1.5mm, F.Cu at (2.80, 61.1)
- added TP108: TestPoint, TestPoint:TestPoint_Pad_D1.5mm, F.Cu at (2.80, 64.7)
- added TP110: TestPoint, TestPoint:TestPoint_Pad_D1.5mm, F.Cu at (6.35, 46.9)
- added TP111: TestPoint, TestPoint:TestPoint_Pad_D1.5mm, F.Cu at (6.35, 50.5)
- added TP112: TestPoint, TestPoint:TestPoint_Pad_D1.5mm, F.Cu at (6.35, 54.0)
- added TP113: TestPoint, TestPoint:TestPoint_Pad_D1.5mm, F.Cu at (6.35, 57.5)
- added TP114: TestPoint, TestPoint:TestPoint_Pad_D1.5mm, F.Cu at (6.35, 61.1)
- added TP115: TestPoint, TestPoint:TestPoint_Pad_D1.5mm, F.Cu at (6.35, 64.7)
- added TP116: TestPoint, TestPoint:TestPoint_Pad_D1.5mm, F.Cu at (9.90, 46.9)
- added TP117: TestPoint, TestPoint:TestPoint_Pad_D1.5mm, F.Cu at (9.90, 50.5)
- added TP118: TestPoint, TestPoint:TestPoint_Pad_D1.5mm, F.Cu at (9.90, 54.0)
- added TP119: TestPoint, TestPoint:TestPoint_Pad_D1.5mm, F.Cu at (9.90, 57.5)
- added TP120: TestPoint, TestPoint:TestPoint_Pad_D1.5mm, F.Cu at (9.90, 61.1)
- added TP121: TestPoint, TestPoint:TestPoint_Pad_D1.5mm, F.Cu at (9.90, 64.7)
- added TP122: TestPoint, TestPoint:TestPoint_Pad_D1.5mm, F.Cu at (13.4, 46.9)
- added TP123: TestPoint, TestPoint:TestPoint_Pad_D1.5mm, F.Cu at (13.4, 50.5)
- added TP124: TestPoint, TestPoint:TestPoint_Pad_D1.5mm, F.Cu at (13.4, 54.0)
- added TP125: TestPoint, TestPoint:TestPoint_Pad_D1.5mm, F.Cu at (13.4, 57.5)
- added TP2: TestPoint, TestPoint:TestPoint_Pad_D1.5mm, F.Cu at (117.9, 160.9)
- added U1: LDI1117-3.3H, Package_TO_SOT_SMD:SOT-223-3_TabPin2, F.Cu at (134.4, 134.5)
- added U2: ESP32-S3-WROOM-1U-N16R2, ESP32-S3-WROOM-1U-N16R2:XCVR_ESP32-S3-WROOM-1U-N16R2, F.Cu at (39.9, 139.4)
- added U3: LMR51610YDBVR, Package_TO_SOT_SMD:SOT-23-6, F.Cu at (122.3, 158.0)
- added U4: STM32G431RBTx, Package_QFP:LQFP-64_10x10mm_P0.5mm, F.Cu at (57.4, 136.2)
- added Y1: 24MHz, Crystal:Crystal_SMD_3225-4Pin_3.2x2.5mm, F.Cu at (52.8, 145.7)
