File: BLDC_DRIVER/BLDC_DRIVER.kicad_pcb (KiCad board)
At the start: 4 copper layers, 100 x 100 mm, 189 parts, among them IC101 DRV8323SRTAR, J1 Terminal, J104 691311400103, J2 Conn_01x03_Pin, J3 Conn_01x03_Pin, J4 Conn_01x06_Pin, Q101 NTMFS4D0N08XT1G, Q102 NTMFS4D0N08XT1G, Q103 NTMFS4D0N08XT1G, Q104 NTMFS4D0N08XT1G, Q105 NTMFS4D0N08XT1G, Q106 NTMFS4D0N08XT1G, SW1 SW_Push, SW2 SW_Push, SW3 SW_Push, SW4 SW_Push, SW5 SW_Push, U1 LDI1117-3.3H, U2 ESP32-S3-WROOM-1U-N16R2, U3 LMR51610YDBVR, U4 STM32G431RBTx, Y1 24MHz

Commit message: mcu&power final layout
Parts:
- removed C103: 100u/200V, EMVY101ARA101MKE0S:CAPAE1300X1400N
- removed F2: 15A, Fuse:Fuse_Blade_ATO_directSolder
- added TP7: TestPoint, TestPoint:TestPoint_Pad_D1.5mm, F.Cu at (184.0, 89.5)
- added TP8: TestPoint, TestPoint:TestPoint_Pad_D1.5mm, F.Cu at (125.9, 80.6)
- added TP9: TestPoint, TestPoint:TestPoint_Pad_D1.5mm, F.Cu at (149.2, 52.2)
- F1: footprint Fuse:Fuse_Blade_ATO_directSolder -> Fuse:Fuse_Blade_Mini_directSolder
- moved F1 84.2 mm to (209.4, 85.8), turned to -90 degrees
- moved R4 59.6 mm to (197.4, 94.4)
- moved R3 59.2 mm to (197.4, 96.2), turned to 180 degrees
- moved U3 58.2 mm to (197.5, 89.1), turned to 90 degrees
- moved D1 55.4 mm to (197.1, 81.9), turned to 90 degrees
- moved R1 55.0 mm to (202.0, 87.2), turned to 90 degrees
- moved R2 54.9 mm to (202.0, 90.8), turned to 90 degrees
- moved TP4 54.3 mm to (193.9, 99.1)
- moved TP3 51.2 mm to (198.5, 100.6)
- moved C6 50.6 mm to (189.5, 94.6), turned to 180 degrees
- moved C5 50.5 mm to (189.5, 92.4), turned to 180 degrees
- moved C4 49.5 mm to (194.7, 90.1), turned to -90 degrees
- moved D4 48.6 mm to (200.1, 108.3), turned to 180 degrees
- moved L1 44.1 mm to (192.1, 84.9), turned to 180 degrees
- moved C105 43.0 mm to (213.6, 41.1)
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Connections:
- R16 pad 1: /MCU/LED3 -> +3.3V
- U2 pad 41_10: (no net) -> GND
- U2 pad 41_11: (no net) -> GND
- U2 pad 41_12: (no net) -> GND
- U2 pad 41_13: (no net) -> GND
- U2 pad 41_14: (no net) -> GND
- U2 pad 41_15: (no net) -> GND
- U2 pad 41_16: (no net) -> GND
- U2 pad 41_17: (no net) -> GND
- U2 pad 41_18: (no net) -> GND
- U2 pad 41_19: (no net) -> GND
- U2 pad 41_20: (no net) -> GND
- U2 pad 41_21: (no net) -> GND
- U4 pad 2: /MCU/FUNC_BTN2 -> unconnected-(U4-PC13-Pad2)
- U4 pad 34: unconnected-(U4-PB12-Pad34) -> /MCU/FUNC_BTN2
- U4 pad 35: /MCU/GL1 -> /MCU/GL3
- U4 pad 37: /MCU/GL3 -> /MCU/GL1
- U4 pad 42: /MCU/GH1 -> /MCU/GH3
- U4 pad 44: /MCU/GH3 -> /MCU/GH1
Routing:
- net /MCU/SDI: track 11.6 -> 68.8 mm, vias 0 -> 2
- net /MCU/SensVC: track 34.6 -> 91.4 mm
- net /MCU/SCLK: track 9.54 -> 63.4 mm, vias 1 -> 2
- net +3.3V: track 202.9 -> 255.7 mm, vias 4 -> 11
- net /MCU/SDO: track 9.42 -> 62.1 mm, vias 1 -> 2
- net /MCU/ENABLE: track 9.79 -> 61.7 mm, vias 1 -> 2
- net /MCU/TEMP_MOSFET: track 113.5 -> 162.4 mm, vias 4 -> 5
- net /MCU/NFAULT: track 10.8 -> 59.2 mm, vias 1 -> 2
- net GND: track 118.6 -> 166.5 mm, vias 33 -> 415
- net /MCU/SensVB: track 32.8 -> 80.5 mm
- net /MCU/NSCS: track 9.67 -> 56.0 mm, vias 1 -> 2
- net /MCU/CAL: track 10.6 -> 56.4 mm, vias 1 -> 2
- net /MCU/SensVN: track 27.5 -> 71.2 mm
- net /MCU/D+: track 0.00 -> 40.3 mm, vias 0 -> 2
- net /MCU/D-: track 0.00 -> 40.3 mm, vias 0 -> 2
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- added copper zone on B.Cu, net GND
- added copper zone on F.Cu, net Net-(J1-Pin_1)

Commit message: finnall layout
Parts:
- added G***: LOGO, LOGO, F.Cu at (142.8, 18.4)
- added G***: LOGO, LOGO, F.Cu at (198.4, 18.4)
- moved TP108 6.20 mm to (147.2, 18.4)
- moved D1 2.63 mm to (195.8, 79.6), turned to 0 degrees
- moved R135 0.20 mm to (153.8, 24.6)
Routing:
- net +48V: track 92.2 -> 100.2 mm, vias 55 -> 98
- net /Motor_driver/SHC: track 136.7 -> 140.8 mm, vias 12 -> 41
- net /Motor_driver/SHA: track 139.1 -> 142.2 mm, vias 10 -> 37
- net /Motor_driver/SHB: track 111.2 -> 114.0 mm, vias 11 -> 20
- net GND: track 166.5 -> 168.1 mm, vias 415 -> 413
- added copper zone on B.Cu, net /Motor_driver/SPC
- added copper zone on B.Cu, net Net-(J1-Pin_1)
Other:
- outline, holes or cut-outs redrawn
- board text added: "BOOT"
- board text added: "Designed by M.Boguski M.Choiński"
- board text added: "EN"
- board text added: "F1"
- board text added: "F2"
- board text added: "G|RX|TX"
- board text added: "RST"
- board text added: "RST|SWO|CLK|GND|DIO|3.3"
