File: BLDC_DRIVER/mcu.kicad_sch (KiCad schematic)
At the start: 48 parts, among them J2 Conn_01x03_Pin, J3 Conn_01x03_Pin, J4 Conn_01x06_Pin, SW1 SW_Push_Dual_x2, SW2 SW_Push_Dual_x2, SW3 SW_Push_Dual_x2, SW4 SW_Push_Dual_x2, SW5 SW_Push_Dual_x2, U2 ESP32-S3-WROOM-1U-N16R2, U4 STM32G431RBTx, Y1 24MHz

Commit message: esp/stm/ldo layout
Parts:
- removed R10, R8: 4.7k, Resistor_SMD:R_0603_1608Metric, symbol Device:R
- removed SW1, SW2, SW3, SW4, SW5: SW_Push_Dual_x2, Button_Switch_SMD:SW_Push_1P1T_NO_CK_KSC7xxJ, symbol Switch:SW_Push_Dual_x2
- added SW1, SW2, SW3, SW4, SW5: SW_Push, Button_Switch_SMD:SW_Tactile_SPST_NO_Straight_CK_PTS636Sx25SMTRLFS, symbol Switch:SW_Push
- renumbered R12 to R10, R13 to R11, R14 to R12, R15 to R13, R16 to R14, R17 to R15, R18 to R16, R19 to R17, R20 to R18, R21 to R19, R22 to R20, R9 to R8, R11 to R9
Connections:
- net BOOT: now also SW4.2
- net ESP_EN: now also SW5.2
- net FUNC_BTN1: now also SW2.2
- net FUNC_BTN2: now also SW3.2
- net NRST: now also SW1.2
- net at R19.1: now also SW4.1
- net at R13.1: now also SW2.1
- net at R14.1: now also SW3.1
- net at R7.1: now also SW1.1
- net at R20.1: now also SW5.1
Other:
- moved on the sheet: R8, R9

Commit message: mcu&power final layout
Connections:
- net +3.3V: now also R16.1
- net FUNC_BTN2: now also U4.34 (PB12); no longer U4.2 (PC13)
- net GH1: now also U4.44 (PA10); no longer U4.42 (PA8)
- net GH3: now also U4.42 (PA8); no longer U4.44 (PA10)
- net GL1: now also U4.37 (PB15); no longer U4.35 (PB13)
- net GL3: now also U4.35 (PB13); no longer U4.37 (PB15)
- net LED3: no longer R16.1
Changed lines of the file:
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@@
-	)
-	(no_connect
-		(at 261.62 107.95)
 	)
 	(no_connect
@@
 	(no_connect
 		(at 152.4 73.66)
+	)
+	(no_connect
+		(at 226.06 90.17)
 	)
 	(no_connect
@@
 		)
 	)
+	(wire
+		(pts
+			(xy 262.89 107.95) (xy 261.62 107.95)
+		)
+		(stroke
+			(width 0)
+			(type default)
+		)
+	)
 	(bus
 		(pts
@@
 	(wire
 		(pts
-			(xy 218.44 90.17) (xy 226.06 90.17)
-		)
-		(stroke
-			(width 0)
-			(type default)
-		)
-	)
-	(wire
-		(pts
 			(xy 58.42 106.68) (xy 60.96 106.68)
 		)
@@
 		(pts
 			(xy 52.07 106.68) (xy 58.42 106.68)
+		)
+		(stroke
+			(width 0)
+			(type default)
+		)
+	)
+	(wire
+		(pts
+			(xy 24.13 152.4) (xy 26.67 152.4)
 		)
 		(stroke
@@
 		)
 	)
-	(label "GL1"
-		(at 261.62 110.49 0)
+	(label "GH3"
+		(at 261.62 54.61 0)
 		(effects
 			(font
@@
 		)
 	)
+	(label "GH1"
+		(at 261.62 59.69 0)
+		(effects
+			(font
+				(size 1.27 1.27)
+			)
+			(justify left bottom)
+		)
+	)
 	(label "SWDIO"
 		(at 40.64 78.74 0)
@@
 		)
 	)
+	(label "GL1"
+		(at 261.62 115.57 0)
+		(effects
+			(font
+				(size 1.27 1.27)
+			)
+			(justify left bottom)
+		)
+	)
 	(label "RX_STM32"
 		(at 90.17 83.82 0)
@@
 		)
 	)
-	(label "GH1"
-		(at 261.62 54.61 0)
-		(effects
-			(font
-				(size 1.27 1.27)
-			)
-			(justify left bottom)
-		)
-	)
 	(label "SWDIO"
 		(at 261.62 67.31 0)
@@
 		)
 	)
-	(label "FUNC_BTN2"
-		(at 218.44 90.17 180)
-		(effects
-			(font
-				(size 1.27 1.27)
-			)
-			(justify right bottom)
-		)
-	)
 	(label "D-"
 		(at 152.4 48.26 0)
@@
 		)
 	)
-	(label "GL3"
-		(at 261.62 115.57 0)
-		(effects
-			(font
-				(size 1.27 1.27)
-			)
-			(justify left bottom)
-		)
-	)
 	(label "LED2"
 		(at 226.06 82.55 180)
@@
 		)
 	)
+	(label "FUNC_BTN2"
+		(at 262.89 107.95 0)
+		(effects
+			(font
+				(size 1.27 1.27)
+			)
+			(justify left bottom)
+		)
+	)
 	(label "ESP_EN"
 		(at 109.22 181.61 0)
@@
 		)
 	)
-	(label "GH3"
-		(at 261.62 59.69 0)
-		(effects
-			(font
-				(size 1.27 1.27)
-			)
-			(justify left bottom)
-		)
-	)
 	(label "RCC_OSC_IN"
 		(at 34.29 106.68 180)
@@
 		)
 	)
-	(label "LED3"
-		(at 26.67 152.4 180)
-		(effects
-			(font
-				(size 1.27 1.27)
-			)
-			(justify right bottom)
-		)
-	)
 	(label "FUNC_BTN1"
 		(at 261.62 100.33 0)
@@
 	(label "GH2"
 		(at 101.6 115.57 0)
+		(effects
+			(font
+				(size 1.27 1.27)
+			)
+			(justify left bottom)
+		)
+	)
+	(label "GL3"
+		(at 261.62 110.49 0)
 		(effects
 			(font
@@
 		)
 	)
+	(symbol
+		(lib_id "power:+3.3V")
+		(at 24.13 152.4 0)
+		(unit 1)
+		(exclude_from_sim no)
+		(in_bom yes)
+		(on_board yes)
+		(dnp no)
+		(property "Reference" "#PWR063"
+			(at 24.13 156.21 0)
+			(effects
+				(font
+					(size 1.27 1.27)
+				)
+				(hide yes)
+			)
+		)
+		(property "Value" "+3.3V"
+			(at 24.13 148.844 0)
+			(effects
+				(font
+					(size 1.27 1.27)
+				)
+			)
+		)
+		(property "Footprint" ""
+			(at 24.13 152.4 0)
+			(effects
+				(font
+					(size 1.27 1.27)
+				)
+				(hide yes)
+			)
+		)
+		(property "Datasheet" ""
+			(at 24.13 152.4 0)
+			(effects
+				(font
+					(size 1.27 1.27)
+				)
+				(hide yes)
+			)
+		)
+		(property "Description" "Power symbol creates a global label with name \"+3.3V\""
+			(at 24.13 152.4 0)
+			(effects
+				(font
+					(size 1.27 1.27)
+				)
+				(hide yes)
+			)
+		)
+		(pin "1"
+		)
+		(instances
+			(project "BLDC_DRIVER"
+				(path "/3fb7c58e-7fa7-4c2f-8afc-969dd7f24a74/3858e4a6-498a-4dbf-a28d-a3d68cd1c461"
+					(reference "#PWR063")
+					(unit 1)
+				)
+			)
+		)
+	)
