File: BLDC_DRIVER/power.kicad_sch (KiCad schematic)
At the start: 27 parts, among them J1 Terminal, U1 LDI1117-3.3H, U3 LMR51610YDBVR

Commit message: esp/stm/ldo layout
Parts:
- C1: footprint EMVY101ARA101MKE0S:CAPAE1300X1400N -> Capacitor_SMD:C_0805_2012Metric_Pad1.18x1.45mm_HandSolder
Changed lines of the file:
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@@
 			)
 		)
-		(property "Footprint" "EMVY101ARA101MKE0S:CAPAE1300X1400N"
+		(property "Footprint" "Capacitor_SMD:C_0805_2012Metric_Pad1.18x1.45mm_HandSolder"
 			(at 40.3352 57.15 0)
 			(effects

Commit message: mcu&power final layout
Parts:
- removed F2: 15A, Fuse:Fuse_Blade_ATO_directSolder, symbol Device:Fuse
- added TP7, TP8, TP9: TestPoint, TestPoint:TestPoint_Pad_D1.5mm, symbol Connector:TestPoint
- F1: footprint Fuse:Fuse_Blade_ATO_directSolder -> Fuse:Fuse_Blade_Mini_directSolder
Connections:
- net GND: now also TP7.1, TP8.1, TP9.1
Other:
- note added: "TEST POINTS GND"
- note removed: "CHOOSE FOTPRINT FOR ELECTROLITIC"
- moved on the sheet: F1
